File: kicad_project-name/kicad_project-name.kicad_pcb (KiCad board)
At the start: 2 copper layers, 0 parts

Commit message: Added configu values for NETs
Other:
- net class USB added: clearance 0.3048, trace_width 0.1524, via_dia 0.6, via_drill 0.3
- net class USB_HS added: clearance 0.6096, trace_width 0.1524, via_dia 0.6, via_drill 0.3
Changed lines of the file:
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@@
+    (uvia_drill 0.1)
+  )
+  (net_class USB ""
+    (clearance 0.3048)
+    (trace_width 0.1524)
+    (via_dia 0.6)
+    (via_drill 0.3)
+    (uvia_dia 0.3)
+    (uvia_drill 0.1)
+  )
+  (net_class USB_HS ""
+    (clearance 0.6096)
+    (trace_width 0.1524)
+    (via_dia 0.6)
+    (via_drill 0.3)
+    (uvia_dia 0.3)
     (uvia_drill 0.1)
   )
